File: prrpls406.kicad_sch (KiCad schematic)
At the start: 52 parts, among them U1001 ATtiny406-M

Commit message: made a new panel
Parts:
- removed D1003, D1007: LED_Small_Filled, JSK:LED_0402_1005Metric, symbol Device:LED_Small_Filled
- removed H1001, H1003, H1004, H1005, H1006, H1008, H1009, H1010, H1012, H1013, H1014, H1015, H1017, H1018, H1019, H1020, H1021, H1022, H1023, H1024, H1026, H1027, H1028, H1030, H1031, H1032, H1033, H1035, H1036: MountingHole, JSK:0.3 npth, symbol Mechanical:MountingHole
- removed H1007, H1016, H1029: MountingHole, JSK:0.5 npth, symbol Mechanical:MountingHole
- removed R1002, R1006: 0, Resistor_SMD:R_0402_1005Metric, symbol Device:R_Small_US
- added D1, D4: LED_Small_Filled, JSK:LED_0402_1005Metric, symbol Device:LED_Small_Filled
- added H1, H2, H3: MountingHole, JSK:0.5 npth, symbol Mechanical:MountingHole
- added R1, R4: 0, JSK:Jumpered_R_0402_1005Metric, symbol Device:R_Small_US
- R2: renamed from R1001; footprint Resistor_SMD:R_0402_1005Metric -> JSK:Jumpered_R_0402_1005Metric
- R3: renamed from R1007; footprint Resistor_SMD:R_0402_1005Metric -> JSK:Jumpered_R_0402_1005Metric
- R5: renamed from R1005; footprint Resistor_SMD:R_0402_1005Metric -> JSK:Jumpered_R_0402_1005Metric
- R6: renamed from R1003; footprint Resistor_SMD:R_0402_1005Metric -> JSK:Jumpered_R_0402_1005Metric
- R7: renamed from R1004; footprint Resistor_SMD:R_0402_1005Metric -> JSK:Jumpered_R_0402_1005Metric
- U1: renamed from U1001; footprint Package_DFN_QFN:VQFN-20-1EP_3x3mm_P0.4mm_EP1.7x1.7mm -> JSK:extra_clearence_VQFN-20-1EP_3x3mm_P0.4mm_EP1.7x1.7mm
- renumbered C1001 to C1, D1002 to D2, D1001 to D3, D1006 to D5, D1005 to D6, D1004 to D7, TP1002 to TP1, TP1004 to TP2, TP1003 to TP3, TP1001 to TP4
Connections:
- net GND: now also U1.8 (PA7), D1.1 (K), D4.1 (K)
- net Serial: now also U1.12 (PB2); no longer U1.20 (PA1)
- net at U1.14 (PB0): now also R7.1
- net at R5.1: now also U1.20 (PA1); no longer U1.1 (PA2)
- net at U1.10 (PB4): now also R1.1
- net at U1.11 (PB3): now also R4.1
- net at U1.15 (PC0): no longer R7.1
- net at U1.16 (PC1): now also R6.1
- net at U1.17 (PC2): no longer R6.1
- new net: D4.2 (A), R4.2
- new net: D1.2 (A), R1.2
Other:
- moved on the sheet: D5, D6, D7, R5, R6, R7

Commit message: submitting
Parts:
- C1: DigiKey PN (none) -> 445-7384-1-ND; LCSC PN (none) -> C3894247; MPN (none) -> C1005X5R1V104K050BB; Manufacturer (none) -> TDK Corporation
- D1, D2, D3, D4, D5, D6, D7: value LED_Small_Filled -> Amber; DigiKey PN (none) -> 3147-B2841UY--20D000414U1930CT-ND; MPN (none) -> B2841UY--20D000414U1930; Manufacturer (none) -> Harvatek Corporation
- U1: DigiKey PN (none) -> ATTINY406-MNRCT-ND; LCSC PN (none) -> C617919; MPN (none) -> ATTINY406-MNR; Manufacturer (none) -> Microchip Technology
