File: programmer/programmer.kicad_pcb (KiCad board)
At the start: 2 copper layers, 28.9 x 13.3 mm, 9 parts, among them J1001 0985-0-15-20-71-14-11-0, J1002 0985-0-15-20-71-14-11-0, J1003 0985-0-15-20-71-14-11-0, J1004 0985-0-15-20-71-14-11-0, J1006 Conn_01x04

Commit message: final update
Other:
- board text added: "WayWayWay"
Changed lines of the file:
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@@
+		)
+	)
+	(gr_text "WayWayWay"
+		(at 131.59 86.24 0)
+		(layer "B.SilkS")
+		(effects
+			(font
+				(size 1 1)
+				(thickness 0.2)
+				(bold yes)
+			)
+			(justify left bottom mirror)
 		)
 	)
